File: logger3.brd (EAGLE design)
At the start: 99 x 44.1 mm, 75 parts, among them IC1 LTC4412, J1 POWER_JACKPTH, Q1 FDN360P, Q2 FDN360P, Q3 2N7002PW, Q4 2N7002PW, U2 FT231X-Q

Commit message: fully routed and ready for check
Parts:
- removed 3.3_SENSE_LT1461: LT1461DHS8-5PBF, LTC_By_element14_Batch_1:SOIC127P600X175-8N
- added 3.3_SENSE: LT1461DHS8-5PBF, LTC_By_element14_Batch_1:SOIC127P600X175-8N
- moved SENSE_CIN 92.7 mm to (71.9, 25.9), turned to 180 degrees
- moved LOGO1 37.7 mm to (54.8, 14.8)
- moved C_LDO_SENSE 33.6 mm to (70.6, 16.3), turned to 0 degrees
- moved U$2 17.2 mm to (68.3, 40.8), turned to 90 degrees
- moved LD0_SD 16.6 mm to (63.1, 34.8)
- moved CLOCK_CIN 16.6 mm to (70.0, 37.5), turned to 0 degrees
- moved C_LDO_SD 16.5 mm to (66.3, 34.8)
- moved C_LDO_CLOCK 16.2 mm to (73.2, 35.0)
- moved CLOCK 16.0 mm to (70.0, 34.8)
- moved SD_CIN 15.1 mm to (63.4, 37.9)
- moved D2 10.2 mm to (50.4, 30.8), turned to 0 degrees
- moved RCKL1 6.29 mm to (72.6, 29.9), turned to 90 degrees
- moved CLOCK_BATT_DECOUP 6.08 mm to (77.6, 25.6), turned to 0 degrees
- moved ADECOUP 5.31 mm to (43.7, 30.9), turned to 180 degrees
- moved CX0 4.85 mm to (60.0, 25.3), turned to 0 degrees
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Connections:
- net +3V3: now also 3.3_SENSE.6, H0.3, H0.5, H3.6; no longer 3.3_SENSE_LT1461.6, H0.2, H0.4, H0.6, H0.8, H3.7
- net 5V: now also H3.7; no longer H3.6
- net A0: now also H0.2; no longer H0.1
- net A1: now also H0.4; no longer H0.3
- net A2: now also H0.6; no longer H0.5
- net A3: now also H0.8; no longer H0.7
- net D4-SENSE_LDO_SWITCH: now also 3.3_SENSE.3; no longer 3.3_SENSE_LT1461.3
- net D7-CS-EXT: now also H3.5; no longer H3.4
- net GND: now also 3.3_SENSE.4, H0.1, H0.7; no longer 3.3_SENSE_LT1461.4
- net VCC: now also 3.3_SENSE.2, H3.4; no longer 3.3_SENSE_LT1461.2, H3.5
Routing:
- net VCC: track 0.00 -> 218.1 mm, vias 0 -> 2
- net +3V3: track 0.00 -> 102.1 mm, vias 0 -> 3
- net VDD: track 0.00 -> 100.1 mm, vias 0 -> 6
- net RESET: track 0.00 -> 72.5 mm, vias 0 -> 2
- net SCL: track 0.00 -> 61.3 mm, vias 0 -> 3
- net CLK: track 0.00 -> 57.7 mm, vias 0 -> 2
- net N$11: track 0.00 -> 54.4 mm, vias 0 -> 2
- net DO: track 0.00 -> 51.3 mm, vias 0 -> 3
- net 5V: track 0.00 -> 50.6 mm, vias 0 -> 1
- net RX-I: track 0.00 -> 49.9 mm, vias 0 -> 2
- net DI: track 0.00 -> 47.0 mm, vias 0 -> 3
- net SDA: track 0.00 -> 45.7 mm, vias 0 -> 3
- net TX-O: track 0.00 -> 42.7 mm, vias 0 -> 2
- net VCL: track 0.00 -> 42.1 mm, vias 0 -> 2
- net N$7: track 0.00 -> 39.4 mm
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