File: logger_2G_GSM.brd (EAGLE design)
At the start: 99 x 44.1 mm, 78 parts, among them IC1 LTC4412, J1 POWER_JACKPTH, Q1 FDN360P, Q2 FDN360P, Q3 2N7002PW, Q4 2N7002PW, U1 DS3231MZ/V+T, U2 FT231X-Q

Commit message: Added JST connector option to logger, started 2G communication
Parts:
- removed C17: 0.1uF, resistor:C0603
- removed C21: 10uF, SparkFun-Passives:EIA3216
- removed CX2, CX3: 33pF, resistor:C0603
- removed D+, D-: 27ohm, rcl:R0603
- removed LSHIFT: 4050D, 40xx:SO16
- added ADC1: (no value), adafruit:1X01-CLEANBIG
- added C2: 1uF, microbuilder:0603-NO
- added C3, C4: 22pF, microbuilder:0603-NO
- added C9: 10uF, microbuilder:0805-NO
- added D3: SMF05C, microbuilder:SOT363
- added D4, D5, D7, D9: 1N4148, microbuilder:SOD-323
- added R6: 10K, microbuilder:0805-NO
- added R9: DNP, microbuilder:0603-NO
- added SJ1: (no value), microbuilder:SOLDERJUMPER_CLOSEDWIRE
- added TP1, TP2, TP3: (no value), microbuilder:TESTPOINT_ROUND_1.5MM
- added U$21: ATSAMD21G18_QFN, microbuilder:TQFN48_7MM
- added U3: SIM808, microbuilder:SIM900_SMT
- added X1: 32.768, adafruit2:XTAL3215
- added X2: 4UCON 20217, microbuilder:4UCONN_20217
- added X3, X4: uFL, microbuilder:U.FL
- added X5, X6: 1x2, con-molex:87758-0216
- added X7: ANT_2450AT18B100, microbuilder:ANT_2450AT18B100
- C1: value 0.1uF -> 10uF; device resistor:C0603 -> microbuilder:_0805MP
- U2: value FT231X-Q -> SIM800H/L; device FT231X:QFN20 -> microbuilder:SIM800L
- moved LED 239.8 mm to (-18.3, -194.4), turned to 0 degrees
- moved ADECOUP 228.0 mm to (-19.1, -189.7), turned to 0 degrees
- moved L_LPF 227.2 mm to (-10.8, -193.7), turned to 0 degrees
- moved CX0 225.6 mm to (-8.76, -189.7)
- moved XTAL 223.9 mm to (-15.0, -182.5)
- moved CX1 223.2 mm to (-3.43, -189.7), turned to 0 degrees
- moved R_LED 220.4 mm to (-7.87, -180.5), turned to 0 degrees
- moved MCU 204.1 mm to (-15.1, -171.3), turned to 0 degrees
- moved C1 181.7 mm to (-18.5, -139.2), turned to 0 degrees
- moved U2 162.5 mm to (-10.4, -119.4), turned to 0 degrees
Connections:
- removed net N$27: RN1.1, U2.17
- removed net N$29: RN1.2, U2.1
- new net !RESET: U$21.40
- new net 1.8V: D3.1, U2.16, U3.P$29, X2.VCC
- new net 2.8V: R6.2, U2.18, U3.P$7
- new net 4_RST: R9.2, U2.49
- new net 5_UART_DTR: D5.C
- new net 6_UART_RTS: D4.C
- new net 7_UART_RI: U2.68
- new net 8_UART_TXD: U2.32
- new net 9_UART_RXD: D9.C
- new net A4: U$21.10
- new net A5: U$21.47
- new net AREF: U$21.4
- new net D+: U$21.34
- new net D-: U$21.33
- new net D0: U$21.16
- new net D1: U$21.15
- new net D10: U$21.27
- new net D11: U$21.25
- new net D12: U$21.28
- new net D13: U$21.26
- new net D2: U$21.23
- new net D3: U$21.14
- new net D5: U$21.24
- new net D6: U$21.29
- new net D7: U$21.30
- new net D8: U$21.11
- new net D9: U$21.12
- new net FM_ANT: TP1.P$1, U2.17
- new net GSM_ANT: U2.40, U3.P$66, X4.3
- new net KEY: D7.C, SJ1.2
- new net MIC1+: U3.P$19
- new net MIC1-: U3.P$20
- new net MIC2+: U2.9, X5.1
- new net MIC2-: U2.10, X5.2
- new net MISO: U$21.21
- new net MOSI: U$21.19
- new net N$18: JP5.VBUS
- new net N$19: C4.1, U$21.2, X1.P$2
- new net NETSTAT: U2.64, U3.P$50
- new net PWRKEY: U3.P$8
- new net PWRSTAT: U2.4, U3.P$49
- new net RI: U3.P$10
- new net RTS: R6.1, U3.P$13
- new net SCK: U$21.20
- new net SD_DO: H3.2, ISP.1, SD.7
- new net SIM808_RST: U3.P$16
- new net SIMCLK: D3.4, U2.55, U3.P$31, X2.CLK
- new net SIMDATA: D3.5, U2.14, U3.P$30, X2.I/O
- new net SIMRST: D3.3, U2.15, U3.P$32, X2.RST
- new net SPEAKER1+: U3.P$21
- new net SPEAKER1-: U3.P$22
- new net SPEAKER2+: U2.51, X6.1
- new net SPEAKER2-: U2.11, X6.2
- new net SWCLK: TP2.P$1, U$21.45
- new net SWDIO: TP3.P$1, U$21.46
- new net UART_DTR: D5.A, U2.69
- new net UART_RTS: D4.A, U2.33
- new net UART_RXD: D9.A, U2.31, U3.P$15
- new net UART_TXD: U3.P$14
- new net VBAT: U2.1, U2.42, U3.P$4, U3.P$5, U3.P$6
- new net VBUS: U2.7, U3.P$25
- new net VDDCORE: C2.1, U$21.43
- new net VRTC: C1.1, C9.1, U2.56, U3.P$17
- net +3V3: now also U$21.17, U$21.36, U$21.44, U$21.6
- net A0: now also U$21.3
- net A1: now also U$21.7
- net A2: now also U$21.8
- net A3: now also U$21.9
- net CLK: no longer LSHIFT.3
- net CS-SD: no longer LSHIFT.7
- net DI: no longer LSHIFT.5
- net DO: no longer H3.2, ISP.1, SD.7
- net DTR: no longer U2.18
- net GND: now also C2.2, C3.2, C4.2, C9.2, D3.2, R9.1, SJ1.1, U$21.18, U$21.35, U$21.42, U$21.5, U$21.THERMAL, U2.2, U2.35, U2.37, U2.38, U2.39, U2.41, U2.43, U2.44, U2.45, U2.57, U2.58, U2.67, U2.71, U2.72, U2.73, U2.76, U2.77, U2.78, U2.79, U2.8, U2.80, U2.81, U2.82, U2.83, U2.84, U2.85, U2.86, U2.87, U2.88, U3.P$1, U3.P$18, U3.P$2, U3.P$28, U3.P$3, U3.P$34, U3.P$36, U3.P$40, U3.P$51, U3.P$52, U3.P$54, U3.P$64, U3.P$65, U3.P$67, U3.P$68, X2.GND, X2.GND@1, X2.GND@2, X2.GND@3, X2.GND@4, X3.1, X3.2, X4.1, X4.2; no longer C17.2, C21.C, CX2.1, CX3.1, LSHIFT.11, LSHIFT.14, LSHIFT.8, LSHIFT.9, U2.13, U2.21, U2.3
- net N$10: now also ADC1.1, U3.P$23; no longer LED1.C, U2.14
- net N$13: now also U2.36, X7.FP; no longer D-.1, U2.9
- net N$16: now also D7.A, U2.48; no longer D+.1, U2.8
- net N$17: now also C3.1, U$21.1, X1.P$1; no longer C1.1, U2.10, U2.11, U2.20
- net N$3: no longer CX3.2, D+.2
- net N$4: no longer CX2.2, D-.2
- net N$6: now also U3.P$35, X3.3; no longer LED2.C, U2.7
- net RX-I: no longer RN1.8
- net SCL: now also U$21.32
- net SDA: now also U$21.31
- net SD_CLK: no longer LSHIFT.2
- net SD_CS: now also U$21.13; no longer LSHIFT.6
- net SD_DI: no longer LSHIFT.4
- net TX-O: no longer RN1.7
- net VDD: no longer LSHIFT.1
- net VUSB: no longer C17.1, C21.A, JP5.VBUS, U2.12
Routing:
- net DO: track 52.1 -> 0.00 mm, vias 3 -> 0
- net SD_DO: track 0.00 -> 51.9 mm, vias 0 -> 3
- net N$10: track 36.5 -> 0.00 mm, vias 2 -> 0
- net N$27: track 28.5 -> 0.00 mm, vias 2 -> 0
- net D9_LED: track 28.4 -> 0.00 mm, vias 2 -> 0
- net CS-SD: track 27.0 -> 0.00 mm, vias 2 -> 0
- net N$29: track 20.2 -> 0.00 mm, vias 2 -> 0
- net N$6: track 20.0 -> 0.00 mm, vias 2 -> 0
- net VUSB: track 31.7 -> 13.2 mm, vias 1 -> 0
- net GND: track 56.5 -> 38.0 mm, vias 38 -> 36
- net N$17: track 18.3 -> 0.00 mm, vias 3 -> 0
- net CLK: track 49.8 -> 33.3 mm
- net AVCC: track 13.0 -> 0.00 mm, vias 2 -> 0
- net X0: track 11.7 -> 0.00 mm
- net X1: track 6.70 -> 0.00 mm
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
Commit message: change 3V3 power supply with jumpers, routing needs finishing
Parts:
- removed ADECOUP: 0.1uF, resistor:C0603
- removed CX0, CX1: 33pF, resistor:C0603
- removed LED: (no value), SparkFun:LED3MM
- removed L_LPF: 10uH, SparkFun:0805
- removed MCU: ATMEGA328P-MU, Atmel_By_element14_Batch_1-00:QFN50P500X500X100-33N
- removed R_LED: 220, resistor:R0603
- removed X2: 4UCON 20217, microbuilder:4UCONN_20217
- removed XTAL: 8MHz, SparkFun:HC49U-V
- added X8: SIM_LOCKAMPHENOL, microbuilder:C707_10M006_512_2
Connections:
- removed net AVCC: ADECOUP.1, L_LPF.2, MCU.18
- removed net CS-SD: MCU.14
- removed net D9_LED: MCU.13, R_LED.1
- removed net DO: MCU.16
- removed net LED+: LED.A, R_LED.2
- removed net X0: CX0.2, MCU.7, XTAL.2
- removed net X1: CX1.2, MCU.8, XTAL.1
- new net N$20: U$21.48
- new net N$21: U$21.39
- net +3V3: no longer MCU.20
- net 1.8V: now also X8.C1; no longer X2.VCC
- net A0: no longer MCU.23
- net A1: no longer MCU.24
- net A2: no longer MCU.25
- net A3: no longer MCU.26
- net A6: no longer MCU.19
- net A7: no longer MCU.22
- net CLK: no longer MCU.17
- net D3-INT1: no longer MCU.1
- net D4-SENSE_LDO_SWITCH: no longer MCU.2
- net D5_MANUAL_LOG: no longer MCU.9
- net D6-CLOCK_3V3_SWITCH: no longer MCU.10
- net D7-CS-EXT: no longer MCU.11
- net D8-SD_3V3_SWITCH: no longer MCU.12
- net DI: no longer MCU.15
- net GND: now also X8.C5; no longer ADECOUP.2, CX0.1, CX1.1, LED.K, MCU.21, MCU.3, MCU.5, X2.GND, X2.GND@1, X2.GND@2, X2.GND@3, X2.GND@4
- net INT0: no longer MCU.32
- net RESET: no longer MCU.29
- net RX-I: no longer MCU.30
- net SCL: no longer MCU.28
- net SDA: no longer MCU.27
- net SIMCLK: now also X8.C3; no longer X2.CLK
- net SIMDATA: now also X8.C7; no longer X2.I/O
- net SIMRST: now also X8.C2; no longer X2.RST
- net TX-O: no longer MCU.31
- net VCC: no longer L_LPF.1, MCU.4, MCU.6
