File: logger_2G_GSM.sch (EAGLE design)
At the start: 78 parts, among them IC1 LTC4412, J1 POWER_JACKPTH, Q1 FDN360P, Q2 FDN360P, Q3 2N7002PW, Q4 2N7002PW, U1 DS3231MZ/V+T, U2 FT231X-Q

Commit message: Added JST connector option to logger, started 2G communication
Parts:
- removed C17: 0.1uF, resistor:C-EUC0603
- removed C21: 10uF, SparkFun-Passives:CAP_POL1206
- removed CX2, CX3: 33pF, resistor:C-EUC0603
- removed D+, D-: 27ohm, rcl:R-US_R0603
- removed LSHIFT: 4050D, 40xx:4050D
- added ADC1: (no value), adafruit:PINHD-1X1CB
- added C2: 1uF, microbuilder:CAP_CERAMIC0603_NO
- added C3, C4: 22pF, microbuilder:CAP_CERAMIC0603_NO
- added C9: 10uF, microbuilder:CAP_CERAMIC0805-NOOUTLINE
- added D3: SMF05C, microbuilder:TVSARRAY_5LANE
- added D4, D5, D7, D9: 1N4148, microbuilder:DIODESOD-323
- added R6: 10K, microbuilder:RESISTOR0805_NOOUTLINE
- added R9: DNP, microbuilder:RESISTOR_0603_NOOUT
- added SJ1: (no value), microbuilder:SOLDERJUMPER_CLOSED
- added TP1, TP2, TP3: (no value), microbuilder:TESTPOINTROUND1.5MM
- added U$21: ATSAMD21G18_QFN, microbuilder:ATSAMD21J_QFN
- added U3: SIM808, microbuilder:GSM_SIM808_LITERAL
- added X1: 32.768, adafruit2:XTAL-3.2X1.5
- added X2: 4UCON 20217, microbuilder:SIM_MICRO
- added X3, X4: uFL, microbuilder:ANTENNA_U.FL
- added X5, X6: 1x2, con-molex:87758-0216
- added X7: ANT_2450AT18B100, microbuilder:ANTENNA_JOHANSON_2450AT18B100
- C1: value 0.1uF -> 10uF; device resistor:C-EUC0603 -> microbuilder:CAP_CERAMIC_0805MP
- U2: value FT231X-Q -> SIM800H/L; device FT231X:FT231X-Q -> microbuilder:GSM_SIM800L
Connections:
- removed net N$27: RN1A.1, U2.TXD
- removed net N$29: RN1B.1, U2.RXD
- new net !RESET: U$21./RESET
- new net 1.8V: D3.C1, U2.VSIM, U3.SIM_VDD, X2.VCC
- new net 2.8V: R6.2, U2.VEXT, U3.VDD_EXT(2.8VOUT)
- new net 4_RST: R9.2, U2.RESET
- new net 5_UART_DTR: D5.C
- new net 6_UART_RTS: D4.C
- new net 7_UART_RI: U2.UART_RI
- new net 8_UART_TXD: U2.UART_TXD
- new net 9_UART_RXD: D9.C
- new net A4: U$21.PA05/EINT5/AIN5/SERCOM0.1
- new net A5: U$21.PB02/I2/AIN10/SERCOM5.0
- new net AREF: U$21.PA03/EINT3/VREFA/AIN1
- new net D+: U$21.PA25/I13/SERCOM3+5.3/D+
- new net D-: U$21.PA24/I12/SERCOM3+5.2/D-
- new net D0: U$21.PA11/I11/AIN19/SERCOM0+2.3/I2SF0
- new net D1: U$21.PA10/I10/AIN18/SERCOM0+2.2/I2SCK
- new net D10: U$21.PA18/I2/SERCOM1+3.2
- new net D11: U$21.PA16/I2C/I0/SERCOM1+3.0
- new net D12: U$21.PA19/I3/SERCOM1+3.3/I2SD0
- new net D13: U$21.PA17/I2C/I1/SERCOM1+3.1
- new net D2: U$21.PA14/I14/SERCOM2+4.2
- new net D3: U$21.PA09/I2C/I9/AIN17/SERCOM0+2.1/I2SMC
- new net D5: U$21.PA15/I15/SERCOM3+4.3
- new net D6: U$21.PA20/I4/SERCOM3+5.2/I2SSC
- new net D7: U$21.PA21/I5/SERCOM3+5.3/I2SFS0
- new net D8: U$21.PA06/EINT6/AIN6/SERCOM0.2
- new net D9: U$21.PA07/I7/AIN7/SERCOM0.3/I2SD0
- new net FM_ANT: TP1.P$1, U2.FM_ANT_P
- new net GSM_ANT: U2.ANT, U3.GSM_RF_IN, X4.SIGNAL
- new net KEY: D7.C, SJ1.2
- new net MIC1+: U3.MIC1P
- new net MIC1-: U3.MIC1N
- new net MIC2+: U2.MIC2P, X5-1.S
- new net MIC2-: U2.MIC2N, X5-2.S
- new net MISO: U$21.PA12/I12/I2C/SERCOM2+4.0
- new net MOSI: U$21.PB10/I10/SERCOM4.2/I2SMC
- new net N$18: JP5.VBUS
- new net N$19: C4.1, U$21.PA01/EINT1/SERCOM1.1, X1.P$2
- new net NETSTAT: U2.NETLIGHT, U3.NETLIGHT
- new net PWRKEY: U3.PWRKEY
- new net PWRSTAT: U2.STATUS, U3.STATUS
- new net RI: U3.RI
- new net RTS: R6.1, U3.RTS
- new net SCK: U$21.PB11/I11/SERCOM4.3/I2SCL
- new net SD_DO: H3.2, ISP.MISO, SD.DATA_OUT
- new net SIM808_RST: U3.RESET
- new net SIMCLK: D3.C3, U2.SIM_CLK, U3.SIM_CLK, X2.CLK
- new net SIMDATA: D3.C4, U2.SIM_DATA, U3.SIM_DATA, X2.DATA
- new net SIMRST: D3.C2, U2.SIM_RST, U3.SIM_RST, X2.RST
- new net SPEAKER1+: U3.SPK1P
- new net SPEAKER1-: U3.SPK1N
- new net SPEAKER2+: U2.SPK2P/8Ω, X6-1.S
- new net SPEAKER2-: U2.SPK2N, X6-2.S
- new net SWCLK: TP2.P$1, U$21.PA30/I10/SECOM1.2/SWCLK
- new net SWDIO: TP3.P$1, U$21.PA31/I11/SECOM1.3/SWDIO
- new net UART_DTR: D5.A, U2.UART_DTR
- new net UART_RTS: D4.A, U2.UART_RTS
- new net UART_RXD: D9.A, U2.UART_RXD, U3.RXD
- new net UART_TXD: U3.TXD
- new net VBAT: U2.VBAT, U3.VBAT@1, U3.VBAT@2, U3.VBAT@3
- new net VDDCORE: C2.1, U$21.VDDCORE
- new net VRTC: C1.1, C9.1, U2.VRTC, U3.VRTC
- net +3V3: now also U$21.VDDA, U$21.VDDIN, U$21.VDDIO
- net A0: now also U$21.PA02/EINT2/AIN0/Y0/VOUT
- net A1: now also U$21.PB08/I8/AIN2/SERCOM4.0
- net A2: now also U$21.PB09/I9/AIN3/SERCOM4.1
- net A3: now also U$21.PA04/EINT4/VREFB/AIN4/SERCOM0.0
- net CLK: no longer LSHIFTA.I
- net CS-SD: no longer LSHIFTC.I
- net DI: no longer LSHIFTB.I
- net DO: no longer H3.2, ISP.MISO, SD.DATA_OUT
- net DTR: no longer U2.DTR#
- net GND: now also C2.2, C3.2, C4.2, C9.2, D3.A, R9.1, SJ1.1, U$21.GND, U$21.GNDA, U2.FM_ANT_N, U2.GND, U3.GND@1, U3.GND@10, U3.GND@11, U3.GND@12, U3.GND@13, U3.GND@14, U3.GND@15, U3.GND@2, U3.GND@3, U3.GND@4, U3.GND@5, U3.GND@6, U3.GND@7, U3.GND@8, U3.GND@9, X2.GND, X3.GND@0, X3.GND@1, X4.GND@0, X4.GND@1; no longer C17.2, C21.-, CX2.1, CX3.1, LSHIFTD.I, LSHIFTE.I, LSHIFTF.I, LSHIFTP.VSS, U2.CTS#, U2.GND@13, U2.GND@21, U2.GND@3
- net N$10: now also ADC1.1, U3.ADC1; no longer LED1.C, U2.CBUS1
- net N$13: now also U2.NC, X7.P$1; no longer D-.1, U2.USBDM
- net N$16: now also D7.A, U2.PWRKEY; no longer D+.1, U2.USBDP
- net N$17: now also C3.1, U$21.PA00/EINT0/SERCOM1.0, X1.P$1; no longer C1.1, U2.3V3OUT, U2.RESET#, U2.VCCIO
- net N$3: no longer CX3.2, D+.2
- net N$4: no longer CX2.2, D-.2
- net N$6: now also U3.GPS_RF_IN, X3.SIGNAL; no longer LED2.C, U2.CBUS2
- net RX-I: no longer RN1A.2
- net SCL: now also U$21.PA23/I2C/I7/SERCOM3+5.1/SOF
- net SDA: now also U$21.PA22/I2C/I6/SERCOM3+5.0
- net SD_CLK: no longer LSHIFTA.O
- net SD_CS: now also U$21.PA08/I2C/AIN16/SERCOM0+2.0/I2SD1; no longer LSHIFTC.O
- net SD_DI: no longer LSHIFTB.O
- net TX-O: no longer RN1B.2
- net VDD: no longer LSHIFTP.VDD
- net VUSB: no longer C17.1, C21.+, JP5.VBUS, U2.VCC
Other:
- note added: "N/C"
- note added: "RXD"
- note added: "RXLED"
- note added: "TXD"
- note added: "TXLED"
- note added: "USBHOSTEN"
- moved on the sheet: ADECOUP, C1, CX0, CX1, LED, LED1, LED2, L_LPF, MCU, RN1C, RN1D, R_LED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

Commit message: change 3V3 power supply with jumpers, routing needs finishing
Parts:
- removed ADECOUP: 0.1uF, resistor:C-EUC0603
- removed CX0, CX1: 33pF, resistor:C-EUC0603
- removed LED: (no value), SparkFun:LED3MM
- removed L_LPF: 10uH, SparkFun:INDUCTOR0805
- removed MCU: ATMEGA328P-MU, Atmel_By_element14_Batch_1-00:ATMEGA328P-MU
- removed R_LED: 220, resistor:R-US_R0603
- removed X2: 4UCON 20217, microbuilder:SIM_MICRO
- removed XTAL: 8MHz, SparkFun:CRYSTALHC49UV
- added X8: SIM_LOCKAMPHENOL, microbuilder:SIM_LOCKAMPHENOL
Connections:
- removed net AVCC: ADECOUP.1, L_LPF.2, MCU.AVCC
- removed net CS-SD: MCU.PB2
- removed net D9_LED: MCU.PB1, R_LED.1
- removed net DO: MCU.PB4
- removed net LED+: LED.A, R_LED.2
- removed net X0: CX0.2, MCU.PB6, XTAL.2
- removed net X1: CX1.2, MCU.PB7, XTAL.1
- new net N$20: U$21.PB03/I3/AIN11/SERCOM5.1
- new net N$21: U$21.PA27/I15
- net +3V3: no longer MCU.AREF
- net 1.8V: now also X8.1; no longer X2.VCC
- net A0: no longer MCU.PC0
- net A1: no longer MCU.PC1
- net A2: no longer MCU.PC2
- net A3: no longer MCU.PC3
- net A6: no longer MCU.ADC6
- net A7: no longer MCU.ADC7
- net CLK: no longer MCU.PB5
- net D3-INT1: no longer MCU.PD3
- net D4-SENSE_LDO_SWITCH: no longer MCU.PD4
- net D5_MANUAL_LOG: no longer MCU.PD5
- net D6-CLOCK_3V3_SWITCH: no longer MCU.PD6
- net D7-CS-EXT: no longer MCU.PD7
- net D8-SD_3V3_SWITCH: no longer MCU.PB0
- net DI: no longer MCU.PB3
- net GND: now also X8.4; no longer ADECOUP.2, CX0.1, CX1.1, LED.C, MCU.GND, MCU.GND_2, MCU.GND_3, X2.GND
- net INT0: no longer MCU.PD2
- net RESET: no longer MCU.PC6
- net RX-I: no longer MCU.PD0
- net SCL: no longer MCU.PC5
- net SDA: no longer MCU.PC4
- net SIMCLK: now also X8.3; no longer X2.CLK
- net SIMDATA: now also X8.6; no longer X2.DATA
- net SIMRST: now also X8.2; no longer X2.RST
- net TX-O: no longer MCU.PD1
- net VCC: no longer L_LPF.1, MCU.VCC, MCU.VCC_2
Other:
- note removed: "RXLED"
- note removed: "TXLED"
- moved on the sheet: A0, A1, A2, A3, A6, A7, C14C, C14D, C15A, C15B, C15C, C15D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
