File: ALog-BottleLogger.sch (EAGLE design)
At the start: 71 parts, among them J1 5.5x2.1mm Barrel, Q1 FDN360P, Q2 FDN360P, Q3 310mA/60V/1.6Ω, Q4 310mA/60V/1.6Ω, U1 DS3231MZ/V+T, U2 FT231X-Q

Commit message: Major revision, 1284P 16 channel 16-bit ADC
Parts:
- removed 3V3: MIC5380_LARGE_PADS, csandell:MIC5380_LARGE_PADS
- removed 5V_CHARGE_PUMP: 5V, ti_by_element14:TPS60150DRVR
- removed A0, A1, A2, A3, A6, A7: (no value), resistor:R-US_0207/10
- removed ADECOUP: 0.1uF, resistor:C-EUC0603
- removed CLOCK_BATT: 3V Backup Battery, awickert:LINX-BAT-HLD-012-SMT-OTL
- removed CLOCK_BATT_DECOUP, COUT1: 0.1uF, rcl:C-EUC0603
- removed CLOCK_BATT_DECOUPLE: 10uF, SparkFun-Passives:CAP_POL1206
- removed CLOCK_CIN1, CLOCK_CIN2, CLOCK_CIN3, COUT: 1uF, rcl:C-EUC0603
- removed CN1: (no value), adafruit:JST_2PIN-THM
- removed CX0, CX1, CX2, CX3: 33pF, resistor:C-EUC0603
- removed C_BOOST_1: 4.7uF, resistor:C-EUC0603
- removed C_BOOST_2, C_BOOST_3: 2.2uF, resistor:C-EUC0603
- removed D+, D-: 27ohm, rcl:R-US_R0603
- removed H0, H1, H3: (no value), SparkFun-Connectors:M10-3.5MM
- removed ISP: AVRISP-6, adafruit:AVRISP-6
- removed JP1, JP2, JP3, JP4: STAND-OFF, SparkFun:STAND-OFF
- removed LED: (no value), SparkFun-LED:LED1206
- removed LED1: Yellow, SparkFun-LED:LED0603
- removed LED2: Blue, SparkFun-LED:LED0603
- removed LOG: LOG, SparkFun-Electromechanical:SWITCH-MOMENTARY-2PTH
- removed LOGO1: OSHW-LOGOM, SparkFun-Aesthetics:OSHW-LOGOM
- removed LSHIFT: 4050D, 40xx:4050D
- removed LTC4412: LTC4412ES6, logger:LTC4412ES6
- removed L_LPF: 10uH, SparkFun:INDUCTOR0805
- removed MCU: ATMEGA328P-MU, Atmel_By_element14_Batch_1-00:ATMEGA328P-MU
- removed MICRO_USB: 10118194-0001LF_LONGER_PADS, 10118194-0001LF:10118194-0001LF_LONGER_PADS
- removed Q1, Q2: FDN360P, transistor-power:FDN360P
- removed Q3, Q4: 310mA/60V/1.6Ω, SparkFun-DiscreteSemi:MOSFET-NCH-2N7002PW
- removed RCKL1, RCLK2: 220, rcl:R-US_R0603
- removed RESET: Reset, SparkFun-Electromechanical:SWITCH-MOMENTARY-2PTH
- removed RN1: 1K, resistor-dil:4R-N0603-ARC
- removed RN2: 3.3K, resistor-dil:4R-N0603-ARC
- removed RSTAT: 470k, rcl:R-US_R0603
- removed R_LED: 220, resistor:R-US_R0603
- removed R_RESET: 10k, rcl:R-US_R0603
- removed U$10: MADE_IN_MN_220, awickert:MADE_IN_MN_220
- removed U2: FT231X-Q, FT231X:FT231X-Q
- removed XTAL: 8MHz, crystal:CRYSTALHC49UP
- added BT1: LINX-BAT-HLD-012-SMT-OTL, awickert:LINX-BAT-HLD-012-SMT-OTL
- added C10, C2, C24: 22uF, rcl:C-EUC0603
- added C11, C5, C6: 0.1uF, rcl:C-EUC0603
- added C12, C13, C16: 10nF, rcl:C-EUC0603
- added C18: .1uF, rcl:C-EUC0603
- added C22, C25: 10uF, rcl:C-EUC0603
- added C23: 10pF, rcl:C-EUC0603
- added C4: 2.2uF, rcl:C-EUC0603
- added C7: 1uF, rcl:C-EUC0603
- added C8, C9: 12nF, rcl:C-EUC0603
- added D3: (no value), SparkFun-LED:LED0603
- added F1, F2: 6V/0.5A, SparkFun-Fuses:PPTC_HALF-AMP
- added IC1: 24AA256SN, microchip:24AA256SN
- added ISP2: AVRISP-6, adafruit:AVRISP-6
- added J10, J2, J5, J8, J9: (no value), SparkFun-Connectors:CONN_10
- added J11, J7: (no value), SparkFun-Connectors:CONN_06SMD-STRAIGHT-FEMALE
- added J3: (no value), SparkFun-Connectors:USB_MICRO-B_SMT
- added J4: (no value), SparkFun-Connectors:JST_2MM_MALE
- added J6: 5.5x2.1mm Barrel, SparkFun-Connectors:POWER_JACKSMD
- added L1: 10uH, Custom:WE-LSQ(INDUCTOR)
- added Q5, Q6, Q7: 4.3A/20V/54mΩ, SparkFun-DiscreteSemi:MOSFET_PCH-IRLML2244
- added Q8, Q9: 220mA/50V/3.5Ω, SparkFun-DiscreteSemi:MOSFET-NCH-BSS138
- added R1: 2M, rcl:R-EU_R0603
- added R10, R11, R12, R20, R21, R22, R42, R43, R44, R45, R46, R47, R7, R8, R9: 10k, rcl:R-EU_R0603
- added R13, R14: FB, rcl:R-EU_R0603
- added R15: 143k, rcl:R-EU_R0603
- added R16: 953k, rcl:R-EU_R0603
- added R2: 383k, rcl:R-EU_R0603
- added R23, R24, R25, R39: 330, rcl:R-EU_R0603
- added R38: 100k, rcl:R-EU_R0603
- added R4, R5: 4.7k, rcl:R-EU_R0603
- added RTC1: DS3231M, SparkFun-Clocks:DS3231M
- added S2, U$1: SKRPABE010, Custom:SKRPABE010
- added U$2: MICROSD, adafruit:MICROSD
- added U$3: TPS6217X, texas:TPS6217X
- added U$5: CM200, Custom:CM200
- added U$6: TPS63061, Custom:TPS306X
- added U$7: LTC2495, linear-technology:LTC2495
- added U$9: 1uH, Custom:WE-MAIA(INDUCTOR)
- added U4: SX1509, SparkFun-IC-Special-Function:SX1509
- C1: value 0.1uF -> 22uF; device resistor:C-EUC0603 -> rcl:C-EUC0603
- C14, C15: device rc-master-smd:CCA_ -> rcl:C-EUC0603
- C17: value 0.1uF -> 10nF; device resistor:C-EUC0603 -> rcl:C-EUC0603
- C21: value 10uF -> 0.1uF; device SparkFun-Passives:CAP_POL1206 -> rcl:C-EUC0603
- D1: value BAT54C -> (none); device semicon-smd-ipc:DIODE_AC-CA_ -> SparkFun-LED:LED0603
- D2: value BAT54 -> (none); device semicon-smd-ipc:DIODE_AC-CA_ -> SparkFun-LED:LED0603
- J1: value 5.5x2.1mm Barrel -> (none); device SparkFun-Connectors:POWER_JACKSMD -> SparkFun-Connectors:CONN_10
- U$8: value ALOG_LOG -> ATMEGA1284P-MU; device awickert:ALOG_LOG -> Atmel_By_element14_Batch_1-00:ATMEGA1284P-MU
- U1: value DS3231MZ/V+T -> ATSAMD21G-A; device Maxim-DS3231MZ_8-SOIC:DS3231MZ/V+T -> SparkFun-IC-Microcontroller:ATSAMD21G-A
Connections:
- removed net +3V3: 3V3.VOUT1, CLOCK_CIN2.1, H0.3, H0.5, H0.9, H1.1, H3.8, MCU.AREF
- removed net A0: A0.2, C14C.1, H0.2, MCU.PC0
- removed net A1: A1.2, C14D.1, H0.4, MCU.PC1
- removed net A2: A2.2, C15A.1, H0.6, MCU.PC2
- removed net A3: A3.2, C15B.1, H0.8, MCU.PC3
- removed net A6: A6.1, C15C.1, H0.10, MCU.ADC6
- removed net A7: A7.1, C15D.1, H1.2, MCU.ADC7
- removed net AVCC: ADECOUP.1, L_LPF.2, MCU.AVCC
- removed net BAT: CLOCK_BATT_DECOUP.1, CLOCK_BATT_DECOUPLE.+, D1.K, U1.VBAT
- removed net CLK: H3.4, ISP.SCK, LSHIFTA.I, MCU.PB5
- removed net CS-SD: LSHIFTC.I, MCU.PB2
- removed net D3-INT1: H1.3, MCU.PD3
- removed net D4-SENSE_LDO_SWITCH: 3V3.EN1, 5V_CHARGE_PUMP.ENA, MCU.PD4
- removed net D5_MANUAL_LOG: D2.A2, MCU.PD5
- removed net D6-EXT: H3.7, MCU.PD6
- removed net D7-CLOCK_SD_SWITCH: 3V3.EN2, MCU.PD7
- removed net D8_LED: MCU.PB0, R_LED.1
- removed net D9-CS-EXT: H3.6, MCU.PB1
- removed net DI: H3.2, ISP.MOSI, LSHIFTB.I, MCU.PB3
- removed net DO: H3.3, ISP.MISO, MCU.PB4, SD.DATA_OUT
- removed net DTR: COUT1.1, U2.DTR#
- removed net INT0: D2.A1, MCU.PD2, U1.*INT/SQW
- removed net LED+: LED.A, R_LED.2
- removed net N$11: D2.K, LOG.2
- removed net N$17: C1.1, U2.3V3OUT, U2.RESET#, U2.VCCIO
- removed net N$2: D-.1, U2.USBDM
- removed net N$29: RN1B.1, U2.RXD
- removed net N$4: CX2.2, D-.2, MICRO_USB.D-
- removed net N$6: LED2.C, U2.CBUS2
- removed net N$67: D1.A2, RCKL1.1
- removed net N$7: LTC4412.STAT, Q2.G, RSTAT.1
- removed net RESET: COUT1.2, ISP.RST, MCU.PC6, RESET.2, R_RESET.1
- removed net RTC_BATT: CLOCK_BATT.+, RCLK2.2
- removed net RX-I: H1.7, MCU.PD0, RN1A.2
- removed net SCL_MCU: MCU.PC5, Q3.D, RN2A.2
- removed net SDA_MCU: MCU.PC4, Q4.D, RN2B.2
- removed net SD_CLK: LSHIFTA.O, SD.SCLK
- removed net SD_DI: LSHIFTB.O, SD.DATA_IN
- removed net TX-O: H1.8, MCU.PD1, RN1B.2
- removed net VBAT: CN1.2, J1.PWR, LTC4412.VIN, Q1.D
- removed net VDD: 3V3.VOUT2, C14B.1, CLOCK_CIN3.1, LSHIFTP.VDD, Q3.G, Q4.G, RN2C.1, RN2D.1, SD.VDD, U1.VCC
- removed net VUSB: C17.1, C21.+, MICRO_USB.VDD, Q2.D, RN1C.2, RN1D.2, U2.VCC
- removed net X0: CX0.2, MCU.PB6, XTAL.2
- removed net X1: CX1.2, MCU.PB7, XTAL.1
- new net 3.3V: C10.1, C11.1, C5.1, C7.1, IC1.VCC, L1.P$2, Q5.S, Q7.S, Q8.G, Q9.G, R1.1, R10.2, R11.2, R12.2, R20.1, R22.1, R23.2, R24.2, R25.2, R4.2, R42.2, R43.2, R5.2, R7.2, RTC1.VCC, U$3.SLEEP, U$3.VOS, U1.VDDANA, U1.VDDIN, U1.VDDIO@17, U1.VDDIO@36, U4.VCC1, U4.VCC2, U4.VDDM
- new net 3.3V_EXT_CTRL: Q5.G, R20.2, U4.I/O[8]
- new net 5V_EXT_CTRL: Q6.G, R21.2, U4.I/O[4]
- new net ADC0: J7.1, J8.2, U$7.CH0
- new net ADC1: J7.2, J8.4, U$7.CH1
- new net ADC10: J5.9, U$7.CH10
- new net ADC11: J5.10, U$7.CH11
- new net ADC2: J7.3, J8.6, U$7.CH2
- new net ADC3: J7.4, J8.8, U$7.CH3
- new net ADC4: J7.5, J8.10, U$7.CH4
- new net ADC5: J7.6, J9.2, U$7.CH5
- new net ADC6: J5.5, U$7.CH6
- new net ADC7: J5.6, U$7.CH7
- new net ADC8: J5.7, U$7.CH8
- new net ADC9: J5.8, U$7.CH9
- new net BATT+: J4.+, J6.PWR, R46.2
- new net EXT_3.3V: F1.2, J10.5, J10.8, J8.3, J8.5, J8.9, J9.1, J9.5
- new net EXT_5V: F2.2, J10.9, J9.4
- new net EXT_D6: J10.7, U4.I/O[10]
- new net EXT_INT: J9.3, U1.PA21(SER5:3+)
- new net GPIO_EXT1: J5.1, U4.I/O[12]
- new net GPIO_EXT2: J5.2, U4.I/O[13]
- new net GPIO_EXT3: J5.3, U4.I/O[14]
- new net GPIO_EXT4: J5.4, U4.I/O[15]
- new net LED1: D1.C, U4.I/O[5]
- new net LED2: D2.C, U4.I/O[6]
- new net LED3: D3.C, U4.I/O[7]
- new net MISO: ISP2.MISO, J10.2, U$2.DATA_OUT, U1.PA12(I2C/SER2:0+)
- new net MOSI: ISP2.MOSI, J10.3, U$2.DATA_IN, U1.PB10(SER4:2+)
- new net MUX_INT: R12.1, U1.PA20(SER5:2+), U4.!INT
- new net N$13: U$7.ADCINN, U$7.MUXOUTN
- new net N$18: F2.1, Q6.D
- new net N$19: U$6.L2, U$9.2
- new net N$20: U$6.L1, U$9.1
- new net N$21: C21.1, U$6.VAUX
- new net N$22: C23.1, R15.2, R16.1, U$6.FB
- new net N$31: BT1.+, RTC1.VBAT
- new net N$32: D1.A, R23.1
- new net N$33: D2.A, R24.1
- new net N$34: D3.A, R25.1
- new net N$44: C12.2, J11.6
- new net N$45: C13.2, J11.5
- new net N$46: C14.2, J11.4
- new net N$47: C15.2, J11.3
- new net N$48: C16.2, J11.2
- new net N$49: C17.2, J11.1
- new net N$50: J3.ID, R38.1, R39.2
- new net N$52: U$7.ADCINP, U$7.MUXOUTP
- new net N$53: R44.1, R45.2, U$7.CH15
- new net N$54: R46.1, R47.1, U$7.CH14
- new net N$56: R11.1, U4.!RESET
- new net RADIO_CS: U1.PA13(I2C/SER2:1+)
- new net RADIO_INT: U1.PA17(I2C/SER1:1+)
- new net RST: ISP2.RST, R7.1, U$1.3, U$1.4, U1.!RESET!
- new net RTC_INT: RTC1.SQW, U1.PA16(I2C/SER1:0+)
- new net RX: U1.PA11(AIN19/SER0:3+)
- new net RX_EXT: J9.7, U1.PA18(SER1:2+)
- new net RX_LED: U1.PB03(AIN11/SER5:1)
- new net SCK: ISP2.SCK, J10.4, U$2.SCLK, U1.PB11(SER4:3+)
- new net SCL_HV: Q9.D, R9.1, U$7.SCL
- new net SDA_HV: Q8.D, R8.1, U$7.SDA
- new net SD_CD: U$2.CARD_DETECT
- new net SD_VCC: Q7.D, U$2.VDD
- new net SD_VCC_CTRL: Q7.G, R22.2, U4.I/O[2]
- new net SPI_EXT_CS1: U4.I/O[11]
- new net SPI_EXT_CS2: J10.6, U4.I/O[9]
- new net TX: U1.PA10(AIN18/SER0:2+)
- new net TX_EXT: J9.8, U1.PA19(SER1:3+)
- new net TX_LED: U1.PA27
- new net USB_D+: R13.2, U1.PA25(SER3:3+)
- new net USB_D-: R14.2, U1.PA24(SER3:2+)
- new net USB_HOST_EN: R39.1, U1.PA28
- net 5V: now also C1.1, C18.1, C2.1, C24.1, C4.1, ISP2.VCC, J3.VBUS, Q6.S, R16.2, R21.1, R38.2, R44.2, R8.2, R9.2, U$3.EN, U$3.VIN, U$6.VOUT, U$7.REF+, U$7.VCC; no longer 5V_CHARGE_PUMP.VOUT, C_BOOST_3.2, H1.4, H3.9
- net GND: now also BT1.-, C10.2, C11.2, C12.1, C13.1, C14.1, C15.1, C16.1, C17.1, C18.2, C2.2, C21.2, C22.2, C23.2, C24.2, C25.2, C4.2, C5.2, C6.2, C7.2, C8.2, C9.2, IC1.A0, IC1.A1, IC1.A2, IC1.GND, IC1.WP, ISP2.GND, J10.1, J10.10, J3.GND, J4.-, J6.GND, J6.GNDBREAK, J8.1, J8.7, J9.6, R15.1, R2.2, R45.1, R47.2, RTC1.GND, S2.3, S2.4, U$1.1, U$1.2, U$2.GND, U$2.GND1, U$2.VSS, U$3.AGND, U$3.BODY, U$3.NC, U$3.PGND, U$6.GND, U$6.PGND, U$6.PS/SYNC, U$7.COM, U$7.GND@1, U$7.GND@2, U$7.GND@3, U$7.GND@4, U$7.GND@5, U$7.GND@6, U$7.GND@7, U$7.GND@8, U$7.REF-, U1.GND@18, U1.GND@35, U1.GND@42, U1.GNDANA, U4.ADDR0, U4.ADDR1, U4.GND; no longer 3V3.GND, 5V_CHARGE_PUMP.EP, 5V_CHARGE_PUMP.GND, A0.1, A1.1, A2.1, A3.1, A6.2, A7.2, ADECOUP.2, C14A.2, C14B.2, C14C.2, C14D.2, C15A.2, C15B.2, C15C.2, C15D.2, C17.2, C21.-, CLOCK_BATT.-, CLOCK_BATT_DECOUP.2, CLOCK_BATT_DECOUPLE.-, CLOCK_CIN1.2, CLOCK_CIN2.2, CLOCK_CIN3.2, CN1.1, COUT.2, CX0.1, CX1.1, CX2.1, CX3.1, C_BOOST_1.1, C_BOOST_3.1, H0.1, H0.7, H1.6, H3.1, H3.10, ISP.GND, J1.GND, J1.GNDBREAK, LED.C, LOG.1, LSHIFTD.I, LSHIFTE.I, LSHIFTF.I, LSHIFTP.VSS, LTC4412.CTL, LTC4412.GND, MCU.EP, MCU.GND, MCU.GND_2, MCU.GND_3, MICRO_USB.GND, RESET.1, SD.COMMON_SW, SD.GND, SD.VSS1, SD.VSS2, U1.GND, U2.CTS#, U2.GND@13, U2.GND@21, U2.GND@3
- net N$1: now also L1.P$1, U$3.SW; no longer D1.A1, RCLK2.1
- net N$10: now also C9.1, U$5.P$1, U1.PA01(XOUT32/SER1:1/TC2:1); no longer LED1.C, U2.CBUS1
- net N$14: now also F1.1, Q5.D; no longer 5V_CHARGE_PUMP.CP+, C_BOOST_2.2
- net N$15: now also J3.D+, R13.1; no longer 5V_CHARGE_PUMP.CP-, C_BOOST_2.1
- net N$16: now also J3.D-, R14.1; no longer D+.1, U2.USBDP
- net N$27: now also U4.OSCIO; no longer RN1A.1, U2.TXD
- net N$3: now also R1.2, R2.1, U$3.FB; no longer CX3.2, D+.2, MICRO_USB.D+
- net N$5: now also R10.1, S2.1, S2.2, U1.PA09(I2C/AIN17/SER0:1+); no longer LED2.A, RN1D.1
- net N$8: now also C6.1, U1.VDDCORE; no longer LTC4412.GATE, Q1.G
- net N$9: now also C8.1, U$5.P$2, U1.PA00(XIN32/SER1:0/TC2:0); no longer LED1.A, RN1C.1
- net SCL: now also IC1.SCL, J9.10, Q9.S, R42.1, R5.1, RTC1.SCL, U1.PA23(I2C/SER3:0+), U4.SCL; no longer H1.10, Q3.S, RN2C.2, U1.SCL
- net SDA: now also IC1.SDA, J9.9, Q8.S, R4.1, R43.1, RTC1.SDA, U1.PA22(I2C/SER3:0+), U4.SDA; no longer H1.9, Q4.S, RN2D.2, U1.SDA
- net SD_CS: now also U$2.CS, U1.PA08(I2C/AIN16/SER0:0+); no longer LSHIFTC.O, SD.CS
- net VCC: now also C22.1, C25.1, U$6.EN, U$6.VIN; no longer 3V3.VIN, 5V_CHARGE_PUMP.VIN, C14A.1, CLOCK_CIN1.1, COUT.1, C_BOOST_1.2, H1.5, H3.5, ISP.VCC, LTC4412.SEN, L_LPF.1, MCU.VCC, MCU.VCC_2, Q1.S, Q2.S, RCKL1.2, RN2A.1, RN2B.1, RSTAT.2, R_RESET.2
Other:
- note added: "2.5v-12v"
- note added: "5v TPS62175"
- note added: "Add fuse?"
- note added: "Add reverse polarity protection?"
- note added: "Analog filter Inductor was ommited since on board analog will not be used"
- note added: "Auxilary I/O connector"
- note added: "Fuse for over current protection on both external lines (0.5A rated)"
- note added: "ICSP"
- note added: "Indicators"
- note added: "Log Switch"
- note added: "NOTE: Add 4 GPIO lines"
- note added: "NOTE: Add bi-directional converters for 5v I2C rail"
- note added: "NOTE: Add control signals!"
- note added: "NOTE: Add ferite beads and/or protection diode?"
- note added: "NOTE: Connect SD_CD to mux input"
- note added: "NOTE: Connect to MUX (open drain)"
- note added: "NOTE: Get info from Ying!"
- note added: "NOTE: Replace footprint!"
- note added: "NOTE: Verify connector!"
- note added: "Note replace buttons!"
- note added: "Power In (From battery)"
- note added: "Resistors divider defaults to 10k Populate secondary slot with alternate resistor and jump to other side to use alternate"
- note added: "SUBNOTE: Fix resistor values"
- note added: "Screw Terminal Connectors"
- note added: "To leave ADCx open (reading from a decive which does not require a resistor divider) leave center tab unjumped"
- note added: "USB Programmer"
- note removed: "1/4"
- note removed: "2.2.0"
- note removed: "2/4"
- note removed: "3/4"
- note removed: "4/4"
- note removed: "ALOG"
- note removed: "ALog data logger by: Andrew Wickert (2011-) and Chad Sandell (2016-) Northern Widget LLC and University of Minnesota"
- note removed: "Andrew Wickert Chad Sandell"
- note removed: "BATTERY_POWER"
- note removed: "I2C BIDIRECTIONAL LEVEL SHIFTER"
- note removed: "MICROCONTROLLER"
- note removed: "POWER MANAGEMENT & DECOUPLING"
- note removed: "REAL TIME CLOCK"
- note removed: "Released under the Creative Commons Attribution Share-Alike 3.0 License http://creativecommons.org/licenses/by-sa/3.0 Design by: Andrew D. Wickert and Chad T. Sandell"
- note removed: "SD CARD AND LEVEL SHIFTER"
- note removed: "USB & ISP"
- note removed: "USER IO & REFERENCE RESISTORS"

Commit message: Work in progress
Parts:
- removed D1, D2, D3: (no value), SparkFun-LED:LED0603
- removed F1, F2: 6V/0.5A, SparkFun-Fuses:PPTC_HALF-AMP
- removed IC1: 24AA256SN, microchip:24AA256SN
- removed R11, R12: 10k, rcl:R-EU_R0603
- removed R2: 383k, rcl:R-EU_R0603
- removed R23, R24, R25, R39: 330, rcl:R-EU_R0603
- removed R38: 100k, rcl:R-EU_R0603
- removed U$2: MICROSD, adafruit:MICROSD
- removed U$5: CM200, Custom:CM200
- removed U4: SX1509, SparkFun-IC-Special-Function:SX1509
- added C19, C20: 0.1uF, rcl:C-EUC0603
- added C26: 1uF, rcl:C-EUC0603
- added C3: 33pF, rcl:C-EUC0603
- added F3, F4: 6V/0.5A, SparkFun-Fuses:PPTC_HALF-AMP
- added J12, J13: (no value), SparkFun-Connectors:M08SMD-STRAIGHT-FEMALE
- added J14, J15, J16: (no value), SparkFun-Connectors:CONN_10
- added J17: (no value), SparkFun-Connectors:M11SMD_NO_HOLES
- added LED: (no value), SparkFun-LED:LED1206
- added Q1, Q2: (no value), crystal:CRYSTALHC49UP
- added R_LED: 220, resistor:R-US_R0603
- added U$4: SKRPABE010, Custom:SKRPABE010
- C11: value 0.1uF -> 33pF
- C4: value 2.2uF -> 10nF; device rcl:C-EUC0603 -> rc-master-smd:CCA_
- J10: device SparkFun-Connectors:CONN_10 -> SparkFun-Connectors:M102MMSMD
- J5, J9: device SparkFun-Connectors:CONN_10 -> SparkFun-Connectors:M08SMD-STRAIGHT-FEMALE
- R1: value 2M -> 10k
Connections:
- removed net EXT_D6: J10.7, U4.I/O[10]
- removed net GPIO_EXT1: J5.1, U4.I/O[12]
- removed net GPIO_EXT2: J5.2, U4.I/O[13]
- removed net GPIO_EXT3: J5.3, U4.I/O[14]
- removed net GPIO_EXT4: J5.4, U4.I/O[15]
- removed net LED1: D1.C, U4.I/O[5]
- removed net LED2: D2.C, U4.I/O[6]
- removed net LED3: D3.C, U4.I/O[7]
- removed net N$14: F1.1, Q5.D
- removed net N$18: F2.1, Q6.D
- removed net N$27: U4.OSCIO
- removed net N$32: D1.A, R23.1
- removed net N$33: D2.A, R24.1
- removed net N$34: D3.A, R25.1
- removed net N$50: J3.ID, R38.1, R39.2
- removed net N$53: R44.1, R45.2, U$7.CH15
- removed net N$54: R46.1, R47.1, U$7.CH14
- removed net N$56: R11.1, U4.!RESET
- removed net SD_CD: U$2.CARD_DETECT
- removed net SPI_EXT_CS1: U4.I/O[11]
- removed net SPI_EXT_CS2: J10.6, U4.I/O[9]
- new net A0: U$8.PA0_(ADC0/PCINT0)
- new net A1: U$8.PA1_(ADC1/PCINT1)
- new net A2: U$8.PA2_(ADC2/PCINT2)
- new net A3: U$8.PA3_(ADC3/PCINT3)
- new net A4: U$8.PA4_(ADC4/PCINT4)
- new net A5: U$8.PA5_(ADC5/PCINT5)
- new net A6: U$8.PA6_(ADC6/PCINT6)
- new net A7: U$8.PA7_(ADC7/PCINT7)
- new net ADC12: J14.7, U$7.CH12
- new net ADC13: J14.6, U$7.CH13
- new net ADC14: J14.2, R46.1, R47.1, U$7.CH14
- new net ADC15: J14.1, R44.1, R45.2, U$7.CH15
- new net EXT_3.3V1: J14.4, J15.4, J16.7, J8.7
- new net EXT_5V1: J14.5, J15.5, J16.8, J8.8
- new net GND1: U$4.1
- new net GND2: C4A.2, C4B.2, C4C.2, C4D.2
- new net GND3: J14.3, J15.3, J16.6, J8.6
- new net LED+: LED.A, R_LED.2
- new net N$17: F3.1, Q5.D
- new net N$2: U$8.~RESET
- new net N$23: F4.1, Q6.D
- new net N$4: U$8.AREF
- new net N$6: C20.1
- new net XTAL2: C11.1, Q2.1, U$8.XTAL2
- net 3.3V: now also C19.1, C26.1, R1.2, R44.2; no longer C11.1, IC1.VCC, R1.1, R11.2, R12.2, R23.2, R24.2, R25.2, U4.VCC1, U4.VCC2, U4.VDDM
- net 3.3V_EXT_CTRL: no longer U4.I/O[8]
- net 5V: no longer C4.1, R38.2, R44.2
- net 5V_EXT_CTRL: no longer U4.I/O[4]
- net ADC0: now also J8.4; no longer J8.2
- net ADC1: now also J8.5; no longer J8.4
- net ADC10: now also J15.2; no longer J5.9
- net ADC11: now also J15.1; no longer J5.10
- net ADC2: now also J8.9; no longer J8.6
- net ADC3: now also J8.10; no longer J8.8
- net ADC4: now also J16.4; no longer J8.10
- net ADC5: now also J16.5; no longer J9.2
- net ADC6: now also J16.9; no longer J5.5
- net ADC7: now also J16.10; no longer J5.6
- net ADC8: now also J15.7; no longer J5.7
- net ADC9: now also J15.6; no longer J5.8
- net EXT_3.3V: now also F3.2, J14.9, J15.9, J16.2, J8.2; no longer F1.2, J10.5, J10.8, J8.3, J8.5, J8.9, J9.1, J9.5
- net EXT_5V: now also F4.2, J14.10, J15.10, J16.3, J8.3; no longer F2.2, J10.9, J9.4
- net EXT_INT: no longer J9.3
- net GND: now also C19.2, C20.2, C26.2, C3.2, J14.8, J15.8, J16.1, SD.COMMON_SW, SD.GND, SD.VSS1, SD.VSS2, U$3.FB, U$8.GND, U$8.GND_2, U$8.GND_3, U$8.GND_4; no longer C4.2, IC1.A0, IC1.A1, IC1.A2, IC1.GND, IC1.WP, J10.1, J10.10, J8.7, J9.6, R2.2, U$2.GND, U$2.GND1, U$2.VSS, U4.ADDR0, U4.ADDR1, U4.GND
- net MISO: no longer J10.2, U$2.DATA_OUT
- net MOSI: no longer J10.3, U$2.DATA_IN
- net MUX_INT: no longer R12.1, U4.!INT
- net N$10: now also Q1.1; no longer U$5.P$1
- net N$3: now also C3.1, Q2.2; no longer R1.2, R2.1, U$3.FB
- net N$9: now also Q1.2; no longer U$5.P$2
- net RST: now also R1.1, U$4.3
- net RX_EXT: no longer J9.7
- net SCK: no longer J10.4, U$2.SCLK
- net SCL: no longer IC1.SCL, J9.10, U4.SCL
- net SDA: no longer IC1.SDA, J9.9, U4.SDA
- net SD_CS: no longer U$2.CS
- net SD_VCC: no longer U$2.VDD
- net SD_VCC_CTRL: no longer U4.I/O[2]
- net TX_EXT: no longer J9.8
- net USB_HOST_EN: no longer R39.1
- net VCC: now also U$8.AVCC, U$8.VCC, U$8.VCC_2, U$8.VCC_3
Other:
- note added: "3.3V TPS62172"
- note added: "NOTE: Why was Bobby measuring the 5V input, should we measure 3.3V?"
- note removed: "5v TPS62175"
- note removed: "Indicators"
- note removed: "NOTE: Connect to MUX (open drain)"
- note removed: "NOTE: Get info from Ying!"
- note removed: "SUBNOTE: Fix resistor values"
- moved on the sheet: C7, C8, C9, J1, J2, J8, Q5, Q6, R20, R21, R44, R45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

Commit message: some progress
Parts:
- removed J10: (no value), SparkFun-Connectors:M102MMSMD
- removed J11, J7: (no value), SparkFun-Connectors:CONN_06SMD-STRAIGHT-FEMALE
- removed J12, J13, J9: (no value), SparkFun-Connectors:M08SMD-STRAIGHT-FEMALE
- removed J17: (no value), SparkFun-Connectors:M11SMD_NO_HOLES
- added C27: 10nF, rc-master-smd:CCA_
- added C28, C29, C30, C31, C32, C33, C34, C35, C36, C37: 10nF, rcl:C-EUC0603
- added C38, C40: 0.1uF, resistor:C-EUC0603
- added C39: 10uF, SparkFun-Passives:CAP_POL1206
- added CX2, CX3: 33pF, resistor:C-EUC0603
- added D+, D-: 27ohm, rcl:R-US_R0603
- added IC2: ATMEGA644M, atmel:ATMEGA644M
- added ISP: AVRISP-6, adafruit:AVRISP-6
- added LED1: Yellow, SparkFun-LED:LED0603
- added LED2: Blue, SparkFun-LED:LED0603
- added MICRO_USB: 10118194-0001LF_LONGER_PADS, 10118194-0001LF:10118194-0001LF_LONGER_PADS
- added R11, R12, R17, R2, R23, R24, R3, R6: 10k, rcl:R-EU_R0603
- added RN1: 1K, resistor-dil:4R-N0603-ARC
- added SJ1, SJ2: SOLDERJUMPER-OLDTRACE, SparkFun-Retired:SOLDERJUMPER-OLDTRACE
- added U2: FT231X-Q, FT231X:FT231X-Q
- J5: device SparkFun-Connectors:M08SMD-STRAIGHT-FEMALE -> SparkFun-Connectors:CONN_10
Connections:
- removed net N$44: C12.2, J11.6
- removed net N$45: C13.2, J11.5
- removed net N$46: C14.2, J11.4
- removed net N$47: C15.2, J11.3
- removed net N$48: C16.2, J11.2
- removed net N$49: C17.2, J11.1
- new net CLK: ISP.SCK
- new net DI: ISP.MOSI
- new net DO: ISP.MISO
- new net DTR: U2.DTR#
- new net GND4: C27A.2, C27B.2, C27C.2, C27D.2
- new net N$14: C4C.2
- new net N$18: R12.1, R17.1, R23.1, R24.1, SJ2.2
- new net N$24: R11.1, R2.1, R3.1, R6.1, SJ1.2
- new net N$25: CX3.2, D+.2, MICRO_USB.D+
- new net N$26: CX2.2, D-.2, MICRO_USB.D-
- new net N$27: RN1A.1, U2.TXD
- new net N$28: D+.1, U2.USBDP
- new net N$29: RN1B.1, U2.RXD
- new net N$30: C40.1, U2.3V3OUT, U2.RESET#, U2.VCCIO
- new net N$32: LED2.A, RN1D.1
- new net N$33: LED2.C, U2.CBUS2
- new net N$34: LED1.A, RN1C.1
- new net N$35: LED1.C, U2.CBUS1
- new net N$36: D-.1, U2.USBDM
- new net RESET: ISP.RST
- new net RX-I: RN1A.2
- new net TX-O: RN1B.2
- new net VUSB: C38.1, C39.+, MICRO_USB.VDD, RN1C.2, RN1D.2, U2.VCC
- net ADC0: now also C12.2, R3.2; no longer J7.1
- net ADC1: now also C13.2, R2.2; no longer J7.2
- net ADC10: now also C32.2
- net ADC11: now also C33.2
- net ADC12: now also C34.2
- net ADC13: now also C35.2
- net ADC14: now also C36.2
- net ADC15: now also C37.2
- net ADC2: now also C14.2, R6.2; no longer J7.3
- net ADC3: now also C15.2, R11.2; no longer J7.4
- net ADC4: now also C16.2, R12.2; no longer J7.5
- net ADC5: now also C17.2, R17.2; no longer J7.6
- net ADC6: now also C28.2, R23.2
- net ADC7: now also C29.2, R24.2
- net ADC8: now also C30.2
- net ADC9: now also C31.2
- net GND: now also C28.1, C29.1, C30.1, C31.1, C32.1, C33.1, C34.1, C35.1, C36.1, C37.1, C38.2, C39.-, C40.2, CX2.1, CX3.1, ISP.GND, MICRO_USB.GND, SJ1.1, SJ2.1, U2.CTS#, U2.GND@13, U2.GND@21, U2.GND@3
- net GND2: no longer C4A.2, C4C.2
- net VCC: now also ISP.VCC
Other:
- note added: "USB & ISP"
- note removed: "Resistors divider defaults to 10k Populate secondary slot with alternate resistor and jump to other side to use alternate"
- note removed: "To leave ADCx open (reading from a decive which does not require a resistor divider) leave center tab unjumped"
- moved on the sheet: C12, C13, C14, C15, C16, C17, C4A, C4B, C4C, C4D

Commit message: more progress
Parts:
- removed BT1: LINX-BAT-HLD-012-SMT-OTL, awickert:LINX-BAT-HLD-012-SMT-OTL
- removed C11, C3: 33pF, rcl:C-EUC0603
- removed C19, C20, C5, C6: 0.1uF, rcl:C-EUC0603
- removed C26, C7: 1uF, rcl:C-EUC0603
- removed C38: 0.1uF, resistor:C-EUC0603
- removed C39: 10uF, SparkFun-Passives:CAP_POL1206
- removed C8, C9: 12nF, rcl:C-EUC0603
- removed ISP: AVRISP-6, adafruit:AVRISP-6
- removed Q1, Q2: (no value), crystal:CRYSTALHC49UP
- removed R10, R7: 10k, rcl:R-EU_R0603
- removed R4, R5: 4.7k, rcl:R-EU_R0603
- removed S2, U$1: SKRPABE010, Custom:SKRPABE010
- removed U$8: ATMEGA1284P-MU, Atmel_By_element14_Batch_1-00:ATMEGA1284P-MU
- removed U1: ATSAMD21G-A, SparkFun-IC-Microcontroller:ATSAMD21G-A
- added C41, C42: 33pF, rcl:C-EUC0603
- added C43: 0.1uF, rcl:C-EUC0603
- added CLOCK_BATT: 3V Backup Battery, awickert:LINX-BAT-HLD-012-SMT-OTL
- added D1, D2: BAT54C, semicon-smd-ipc:DIODE_AC-CA_
- added Q3: (no value), crystal:CRYSTALHC49UP
- added R18, R19: 10k, rcl:R-EU_R0603
- added RCKL2, RCLK1: 220, rcl:R-US_R0603
- added S1: SKRPABE010, Custom:SKRPABE010
Connections:
- removed net A0: U$8.PA0_(ADC0/PCINT0)
- removed net A1: U$8.PA1_(ADC1/PCINT1)
- removed net A2: U$8.PA2_(ADC2/PCINT2)
- removed net A3: U$8.PA3_(ADC3/PCINT3)
- removed net A4: U$8.PA4_(ADC4/PCINT4)
- removed net A5: U$8.PA5_(ADC5/PCINT5)
- removed net A6: U$8.PA6_(ADC6/PCINT6)
- removed net A7: U$8.PA7_(ADC7/PCINT7)
- removed net CLK: ISP.SCK
- removed net DI: ISP.MOSI
- removed net DO: ISP.MISO
- removed net EXT_INT: U1.PA21(SER5:3+)
- removed net GND1: U$4.1
- removed net MUX_INT: U1.PA20(SER5:2+)
- removed net N$10: C9.1, Q1.1, U1.PA01(XOUT32/SER1:1/TC2:1)
- removed net N$2: U$8.~RESET
- removed net N$3: C3.1, Q2.2
- removed net N$4: U$8.AREF
- removed net N$5: R10.1, S2.1, S2.2, U1.PA09(I2C/AIN17/SER0:1+)
- removed net N$6: C20.1
- removed net N$8: C6.1, U1.VDDCORE
- removed net N$9: C8.1, Q1.2, U1.PA00(XIN32/SER1:0/TC2:0)
- removed net RADIO_CS: U1.PA13(I2C/SER2:1+)
- removed net RADIO_INT: U1.PA17(I2C/SER1:1+)
- removed net RESET: ISP.RST
- removed net RX: U1.PA11(AIN19/SER0:3+)
- removed net RX-I: RN1A.2
- removed net RX_EXT: U1.PA18(SER1:2+)
- removed net RX_LED: U1.PB03(AIN11/SER5:1)
- removed net TX: U1.PA10(AIN18/SER0:2+)
- removed net TX-O: RN1B.2
- removed net TX_EXT: U1.PA19(SER1:3+)
- removed net TX_LED: U1.PA27
- removed net USB_HOST_EN: U1.PA28
- removed net VCC: C22.1, C25.1, ISP.VCC, U$6.EN, U$6.VIN, U$8.AVCC, U$8.VCC, U$8.VCC_2, U$8.VCC_3
- new net +3V3: C10.1, IC2.AREF, IC2.AVCC, IC2.VCC, IC2.VCC@1, IC2.VCC@2, ISP2.VCC, L1.P$2, Q8.G, Q9.G, R1.2, R42.2, R43.2, RCKL2.2, U$3.SLEEP, U$3.VOS
- new net +5V: C1.1, C2.1, C24.1, MICRO_USB.VDD, R16.2, U$3.EN, U$3.VIN, U$6.VOUT, U2.VCC
- new net ADC16: IC2.(PCINT7/ADC7)PA7, R18.1, R19.1
- new net AIN1: IC2.(PCINT11/OC0A/AIN1)PB3
- new net CLKO/T1: IC2.(PCINT9/CLKO/T1)PB1
- new net INT2: IC2.(PCINT10/INT2/AIN0)PB2
- new net LED: IC2.(PCINT31/OC2A)PD7, R_LED.1
- new net MANUAL_LOG: D1.A2
- new net MCU_ADC0: IC2.(PCINT0/ADC0)PA0
- new net MCU_ADC1: IC2.(PCINT1/ADC1)PA1
- new net MCU_ADC2: IC2.(PCINT2/ADC2)PA2
- new net MCU_ADC3: IC2.(PCINT3/ADC3)PA3
- new net MCU_ADC4: IC2.(PCINT4/ADC4)PA4
- new net MCU_ADC5: IC2.(PCINT5/ADC5)PA5
- new net MCU_ADC6: IC2.(PCINT6/ADC6)PA6
- new net N$37: D2.K, RTC1.VBAT
- new net N$38: D2.A1, RCLK1.1
- new net N$39: D1.K, S1.1, S1.2
- new net N$56: IC2.(PCINT22/TOSC1)PC6
- new net RTC_BATT: CLOCK_BATT.+, RCLK1.2
- new net RX/INT0: IC2.(PCINT26/INT0)PD2
- new net RX_USB: IC2.(PCINT24/RXD0)PD0, RN1A.2
- new net SS: IC2.(PCINT12/OC0B/!SS!)PB4
- new net TCK: IC2.(PCINT18/TCK)PC2
- new net TDI: IC2.(PCINT21/TDI)PC5
- new net TDO: IC2.(PCINT20/TDO)PC4
- new net TMS: IC2.(PCINT19/TMS)PC3
- new net TX/INT1: IC2.(PCINT27/INT1)PD3
- new net TX_USB: IC2.(PCINT25/TXD0)PD1, RN1B.2
- new net XCK0/T0: IC2.(PCINT8/XCK0/T0)PB0
- new net XTAL1: C42.1, IC2.XTAL1, Q3.1
- net 3.3V: no longer C10.1, C19.1, C26.1, C5.1, C7.1, L1.P$2, Q8.G, Q9.G, R1.2, R10.2, R4.2, R42.2, R43.2, R5.2, R7.2, U$3.SLEEP, U$3.VOS, U1.VDDANA, U1.VDDIN, U1.VDDIO@17, U1.VDDIO@36
- net 3.3V_EXT_CTRL: now also IC2.(PCINT30/OC2B/ICP)PD6
- net 5V: no longer C1.1, C2.1, C24.1, ISP2.VCC, R16.2, U$3.EN, U$3.VIN, U$6.VOUT
- net 5V_EXT_CTRL: now also IC2.(PCINT29/OC1A)PD5
- net BATT+: now also C22.1, C25.1, R18.2, U$6.EN, U$6.VIN
- net GND: now also C41.2, C42.2, C43.2, CLOCK_BATT.-, IC2.EXP, IC2.GND, IC2.GND@1, IC2.GND@2, IC2.GND@3, LED.C, R19.2, S1.3, S1.4, U$4.1, U$4.2; no longer BT1.-, C11.2, C19.2, C20.2, C26.2, C3.2, C38.2, C39.-, C5.2, C6.2, C7.2, C8.2, C9.2, ISP.GND, S2.3, S2.4, U$1.1, U$1.2, U$8.GND, U$8.GND_2, U$8.GND_3, U$8.GND_4, U1.GND@18, U1.GND@35, U1.GND@42, U1.GNDANA
- net MISO: now also IC2.(PCINT14/MISO)PB6, SD.DATA_OUT; no longer U1.PA12(I2C/SER2:0+)
- net MOSI: now also IC2.(PCINT13/MOSI)PB5, SD.DATA_IN; no longer U1.PB10(SER4:2+)
- net N$31: now also D2.A2, RCKL2.1; no longer BT1.+, RTC1.VBAT
- net RST: now also C43.1, IC2.RESET, U$4.4; no longer R7.1, U$1.3, U$1.4, U1.!RESET!
- net RTC_INT: now also D1.A1; no longer U1.PA16(I2C/SER1:0+)
- net SCK: now also IC2.(PCINT15/SCK)PB7, SD.SCLK; no longer U1.PB11(SER4:3+)
- net SCL: now also IC2.(PCINT16/SCL)PC0; no longer R5.1, U1.PA23(I2C/SER3:0+)
- net SDA: now also IC2.(PCINT17/SDA)PC1; no longer R4.1, U1.PA22(I2C/SER3:0+)
- net SD_CS: now also SD.CS; no longer U1.PA08(I2C/AIN16/SER0:0+)
- net SD_VCC: now also SD.VDD
- net SD_VCC_CTRL: now also IC2.(PCINT28/OC1B)PD4
- net USB_D+: no longer U1.PA25(SER3:3+)
- net USB_D-: no longer U1.PA24(SER3:2+)
- net VUSB: no longer C38.1, C39.+, MICRO_USB.VDD, U2.VCC
- net XTAL2: now also C41.1, IC2.XTAL2, Q3.2; no longer C11.1, Q2.1, U$8.XTAL2
Other:
- note added: "Adjust resistors for 3.3V ADC"
- note added: "NOTE: Add precision voltage source, move batt measurement to MCU ADC."
- note removed: "Analog filter Inductor was ommited since on board analog will not be used"
- note removed: "NOTE: Add bi-directional converters for 5v I2C rail"
- note removed: "NOTE: Add control signals!"
- note removed: "NOTE: Connect SD_CD to mux input"
- note removed: "NOTE: Replace footprint!"
- note removed: "NOTE: Why was Bobby measuring the 5V input, should we measure 3.3V?"
- note removed: "Note replace buttons!"

Commit message: progress
Parts:
- removed J3: (no value), SparkFun-Connectors:USB_MICRO-B_SMT
- removed R13, R14: FB, rcl:R-EU_R0603
- removed R46, R47: 10k, rcl:R-EU_R0603
- added Q1, Q4: 220mA/50V/3.5Ω, SparkFun-DiscreteSemi:MOSFET-NCH-BSS138
- added R5: 10k, rcl:R-EU_R0603
- added U$2: MAX6070, bschulz:MAX6070
Connections:
- removed net 3.3V: Q5.S, Q7.S, R20.1, R22.1, R44.2, RTC1.VCC
- removed net USB_D+: R13.2
- removed net USB_D-: R14.2
- new net +3V2: Q4.G
- new net N$10: U$2.OUTF
- new net N$40: U$2.FILT
- new net N$41: U$2.EN
- new net N$9: U$2.GND
- new net USB_STATUS: MICRO_USB.ID
- net +3V3: now also Q1.G, Q5.S, Q7.S, R20.1, R22.1, R44.2, R5.2, RTC1.VCC
- net +5V: now also C18.1, Q6.S, R21.1, R8.2, R9.2, U$7.VCC
- net 5V: no longer C18.1, J3.VBUS, Q6.S, R21.1, R8.2, R9.2, U$7.VCC
- net 5V_EXT_CTRL: now also Q1.S, R5.1; no longer Q6.G, R21.2
- net ADC14: no longer R46.1, R47.1
- net BATT+: no longer R46.2
- net GND: no longer J3.GND, R47.2
- net N$15: now also U$2.OUTS; no longer J3.D+, R13.1
- net N$16: now also U$2.VIN; no longer J3.D-, R14.1
- net SDA_HV: now also Q1.D, Q6.G, R21.2
Other:
- note added: "Add Mosphet control for FTDI"
- note removed: "Add fuse?"
- note removed: "NOTE: Add ferite beads and/or protection diode?"
- note removed: "NOTE: Add precision voltage source, move batt measurement to MCU ADC."
- note removed: "NOTE: Verify connector!"
- note removed: "USB & ISP"
- note removed: "USB Programmer"
- moved on the sheet: MICRO_USB, R8, R9
